Commit message: Added assets to use

File: assets/example-robot-data/end_effectors/robotiq/urdf/robotiq_2f_85_gripper.urdf (robot description, URDF)
Before this commit: robot robotiq_gripper, 10 links, 9 joints
Joints:
- joint robotiq_85_left_finger_tip_joint: type continuous -> revolute
- joint robotiq_85_left_inner_knuckle_joint: type continuous -> revolute
- joint robotiq_85_right_finger_tip_joint: type continuous -> revolute
- joint robotiq_85_right_inner_knuckle_joint: type continuous -> revolute
